File: pcb/Telefunken_Digitale_Electronic_101/buttons.kicad_sch (KiCad schematic)
At the start: 7 parts, among them J1 Conn_01x02_Socket, J2 Conn_01x02_Socket, J3 Conn_01x02_Socket, J4 Conn_01x02_Socket, J5 Conn_01x02_Socket, SW1 SW_Push, SW2 SW_Push

Commit message: SCH and PCB: reannotated everything
Parts:
- renumbered J1 to J4, J2 to J5, J3 to J6, J4 to J7, J5 to J8
Changed lines of the file:
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@@
 		(in_pos_files yes)
 		(dnp no)
-		(property "Reference" "J2"
+		(property "Reference" "J5"
 			(at 66.04 46.9899 0)
 			(hide yes)
@@
 			(project "Telefunken_Digitale_Electronic_101"
 				(path "/df1af5ff-c8b9-4769-9610-ead9e11e7e65/d38ac94e-1578-41e7-bfce-23ec2afd3398"
-					(reference "J2")
+					(reference "J5")
 					(unit 1)
 				)
@@
 		(in_pos_files yes)
 		(dnp no)
-		(property "Reference" "J5"
+		(property "Reference" "J8"
 			(at 119.38 66.0399 0)
 			(hide yes)
@@
 			(project "Telefunken_Digitale_Electronic_101"
 				(path "/df1af5ff-c8b9-4769-9610-ead9e11e7e65/d38ac94e-1578-41e7-bfce-23ec2afd3398"
-					(reference "J5")
+					(reference "J8")
 					(unit 1)
 				)
@@
 		(in_pos_files yes)
 		(dnp no)
-		(property "Reference" "J1"
+		(property "Reference" "J4"
 			(at 66.04 36.8299 0)
 			(hide yes)
@@
 			(project "Telefunken_Digitale_Electronic_101"
 				(path "/df1af5ff-c8b9-4769-9610-ead9e11e7e65/d38ac94e-1578-41e7-bfce-23ec2afd3398"
-					(reference "J1")
+					(reference "J4")
 					(unit 1)
 				)
@@
 		(in_pos_files yes)
 		(dnp no)
-		(property "Reference" "J4"
+		(property "Reference" "J7"
 			(at 66.04 68.5799 0)
 			(hide yes)
@@
 			(project "Telefunken_Digitale_Electronic_101"
 				(path "/df1af5ff-c8b9-4769-9610-ead9e11e7e65/d38ac94e-1578-41e7-bfce-23ec2afd3398"
-					(reference "J4")
+					(reference "J7")
 					(unit 1)
 				)
@@
 		(in_pos_files yes)
 		(dnp no)
-		(property "Reference" "J3"
+		(property "Reference" "J6"
 			(at 66.04 59.6899 0)
 			(hide yes)
@@
 			(project "Telefunken_Digitale_Electronic_101"
 				(path "/df1af5ff-c8b9-4769-9610-ead9e11e7e65/d38ac94e-1578-41e7-bfce-23ec2afd3398"
-					(reference "J3")
+					(reference "J6")
 					(unit 1)
 				)
