File: pcb/Telefunken_Digitale_Electronic_101/buttons.kicad_sch (KiCad schematic)
At the start: 7 parts, among them J4 Conn_01x02_Socket, J5 Conn_01x02_Socket, J6 Conn_01x02_Socket, J7 Conn_01x02_Socket, J8 Conn_01x02_Socket, SW1 SW_Push, SW2 SW_Push

Commit message: SCH and PCB - buttons: added proper switches that will be used
Parts:
- SW1, SW2: footprint Button_Switch_THT:SW_PUSH_6mm_H4.3mm -> RadioWecker:TACT_SWITCH_3.2X4.2X2.5MM
Changed lines of the file:
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@@
 			)
 		)
-		(property "Footprint" "Button_Switch_THT:SW_PUSH_6mm_H4.3mm"
+		(property "Footprint" "RadioWecker:TACT_SWITCH_3.2X4.2X2.5MM"
 			(at 116.84 34.29 0)
 			(hide yes)
@@
 			)
 		)
-		(property "Footprint" "Button_Switch_THT:SW_PUSH_6mm_H4.3mm"
+		(property "Footprint" "RadioWecker:TACT_SWITCH_3.2X4.2X2.5MM"
 			(at 116.84 46.99 0)
 			(hide yes)
