File: pcb/Telefunken_Digitale_Electronic_101/display.kicad_sch (KiCad schematic)
At the start: 8 parts, among them U1 TM1637_SOP20

Commit message: SCH - display: name under Name
Parts:
- DISPLAY1: Name (none) -> DISPLAY
Changed lines of the file:
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@@
 		(in_pos_files yes)
 		(dnp no)
-		(fields_autoplaced yes)
 		(property "Reference" "DISPLAY1"
 			(at 227.33 93.98 0)
+			(hide yes)
 			(show_name no)
 			(do_not_autoplace no)
@@
 			(show_name no)
 			(do_not_autoplace no)
+			(effects
+				(font
+					(size 1.27 1.27)
+				)
+			)
+		)
+		(property "Name" "DISPLAY"
+			(at 206.502 123.952 0)
+			(show_name no)
+			(do_not_autoplace no)

Commit message: SCH - buttons, display and interface: TM1637 can read the buttons (saves many resistors, caps and connectors)
Connections:
- net BUTTONS_GRID4: now reaches DISPLAY1.10 (f), U1.7 (SEG6/KS6)
- net BUTTONS_GRID1: now reaches DISPLAY1.11 (a), U1.2 (SEG1/KS1)
- net BUTTONS_GRID3: now reaches DISPLAY1.4 (c), U1.4 (SEG3/KS3)
- net BUTTONS_GRID2: now reaches DISPLAY1.7 (b), U1.3 (SEG2/KS2)
- net BUTTONS_K1: now reaches U1.19 (K1)
- net BUTTONS_K2: now reaches U1.20 (K2)
- no-connect marks 4 -> 2
Changed lines of the file:
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@@
 		(at 168.91 93.98)
 	)
-	(no_connect
-		(at 133.35 101.6)
-	)
-	(no_connect
-		(at 133.35 104.14)
+	(wire
+		(pts
+			(xy 130.81 101.6) (xy 133.35 101.6)
+		)
+		(stroke
+			(width 0)
+			(type default)
+		)
 	)
 	(wire
@@
 		(pts
 			(xy 168.91 116.84) (xy 199.39 116.84)
+		)
+		(stroke
+			(width 0)
+			(type default)
+		)
+	)
+	(wire
+		(pts
+			(xy 130.81 104.14) (xy 133.35 104.14)
 		)
 		(stroke
@@
 		)
 	)
+	(label "KS3"
+		(at 168.91 106.68 0)
+		(effects
+			(font
+				(size 1.27 1.27)
+			)
+			(justify left bottom)
+		)
+	)
+	(label "KS6"
+		(at 168.91 114.3 0)
+		(effects
+			(font
+				(size 1.27 1.27)
+			)
+			(justify left bottom)
+		)
+	)
+	(label "K2"
+		(at 53.34 97.79 0)
+		(effects
+			(font
+				(size 1.27 1.27)
+			)
+			(justify left bottom)
+		)
+	)
 	(label "DIO"
 		(at 53.34 71.12 0)
@@
 		)
 	)
+	(label "KS2"
+		(at 53.34 87.63 0)
+		(effects
+			(font
+				(size 1.27 1.27)
+			)
+			(justify left bottom)
+		)
+	)
+	(label "KS2"
+		(at 168.91 104.14 0)
+		(effects
+			(font
+				(size 1.27 1.27)
+			)
+			(justify left bottom)
+		)
+	)
+	(label "K2"
+		(at 130.81 104.14 0)
+		(effects
+			(font
+				(size 1.27 1.27)
+			)
+			(justify left bottom)
+		)
+	)
 	(label "CLK"
 		(at 101.6 83.82 0)
@@
 		)
 	)
+	(label "KS3"
+		(at 53.34 90.17 0)
+		(effects
+			(font
+				(size 1.27 1.27)
+			)
+			(justify left bottom)
+		)
+	)
 	(label "CLK"
 		(at 53.34 68.58 0)
@@
 			)
 			(justify left bottom)
+		)
+	)
+	(label "KS1"
+		(at 53.34 85.09 0)
+		(effects
+			(font
+				(size 1.27 1.27)
+			)
+			(justify left bottom)
+		)
+	)
+	(label "KS6"
+		(at 53.34 92.71 0)
+		(effects
+			(font
+				(size 1.27 1.27)
+			)
+			(justify left bottom)
+		)
+	)
+	(label "K1"
+		(at 53.34 95.25 0)
+		(effects
+			(font
+				(size 1.27 1.27)
+			)
+			(justify left bottom)
+		)
+	)
+	(label "KS1"
+		(at 168.91 101.6 0)
+		(effects
+			(font
+				(size 1.27 1.27)
+			)
+			(justify left bottom)
+		)
+	)
+	(label "K1"
+		(at 130.81 101.6 0)
+		(effects
+			(font
+				(size 1.27 1.27)
+			)
+			(justify left bottom)
+		)
+	)
+	(hierarchical_label "BUTTONS_K1"
+		(shape input)
+		(at 53.34 95.25 180)
+		(effects
+			(font
+				(size 1.27 1.27)
+			)
+			(justify right)
 		)
 	)
@@
 		)
 	)
+	(hierarchical_label "BUTTONS_GRID4"
+		(shape output)
+		(at 53.34 92.71 180)
+		(effects
+			(font
+				(size 1.27 1.27)
+			)
+			(justify right)
+		)
+	)
 	(hierarchical_label "GND"
 		(shape bidirectional)
@@
 		)
 	)
+	(hierarchical_label "BUTTONS_GRID2"
+		(shape output)
+		(at 53.34 87.63 180)
+		(effects
+			(font
+				(size 1.27 1.27)
+			)
+			(justify right)
+		)
+	)
+	(hierarchical_label "BUTTONS_GRID1"
+		(shape output)
+		(at 53.34 85.09 180)
+		(effects
+			(font
+				(size 1.27 1.27)
+			)
+			(justify right)
+		)
+	)
 	(hierarchical_label "VCC"
 		(shape bidirectional)
@@
 		(effects
 			(font
+				(size 1.27 1.27)
+			)
+			(justify right)
+		)
+	)
+	(hierarchical_label "BUTTONS_GRID3"
+		(shape output)
+		(at 53.34 90.17 180)
+		(effects
+			(font
+				(size 1.27 1.27)
+			)
+			(justify right)
+		)
+	)
+	(hierarchical_label "BUTTONS_K2"
+		(shape input)
+		(at 53.34 97.79 180)
+		(effects
+			(font

Commit message: SCH and PCB: reannotated everything
Parts:
- renumbered C1 to C5, C2 to C6, C3 to C7, C4 to C8, R1 to R3, R2 to R4, U1 to U2
Changed lines of the file:
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@@
 		(dnp no)
 		(fields_autoplaced yes)
-		(property "Reference" "#PWR03"
+		(property "Reference" "#PWR018"
 			(at 124.46 85.09 0)
 			(hide yes)
@@
 			(project "Telefunken_Digitale_Electronic_101"
 				(path "/df1af5ff-c8b9-4769-9610-ead9e11e7e65/ef6275f4-75ba-4006-a847-a151b9f8c4ad"
-					(reference "#PWR03")
+					(reference "#PWR018")
 					(unit 1)
 				)
@@
 		(dnp no)
 		(fields_autoplaced yes)
-		(property "Reference" "#PWR028"
+		(property "Reference" "#PWR015"
 			(at 57.15 64.77 0)
 			(hide yes)
@@
 			(project "Telefunken_Digitale_Electronic_101"
 				(path "/df1af5ff-c8b9-4769-9610-ead9e11e7e65/ef6275f4-75ba-4006-a847-a151b9f8c4ad"
-					(reference "#PWR028")
+					(reference "#PWR015")
 					(unit 1)
 				)
@@
 		(dnp no)
 		(fields_autoplaced yes)
-		(property "Reference" "C3"
+		(property "Reference" "C7"
 			(at 180.34 72.3899 0)
 			(show_name no)
@@
 			(project "Telefunken_Digitale_Electronic_101"
 				(path "/df1af5ff-c8b9-4769-9610-ead9e11e7e65/ef6275f4-75ba-4006-a847-a151b9f8c4ad"
-					(reference "C3")
+					(reference "C7")
 					(unit 1)
 				)
@@
 		(dnp no)
 		(fields_autoplaced yes)
-		(property "Reference" "U1"
+		(property "Reference" "U2"
 			(at 151.13 71.12 0)
 			(show_name no)
@@
 			(project "Telefunken_Digitale_Electronic_101"
 				(path "/df1af5ff-c8b9-4769-9610-ead9e11e7e65/ef6275f4-75ba-4006-a847-a151b9f8c4ad"
-					(reference "U1")
+					(reference "U2")
 					(unit 1)
 				)
@@
 		(in_pos_files yes)
 		(dnp no)
-		(property "Reference" "C1"
+		(property "Reference" "C5"
 			(at 119.634 87.884 0)
 			(show_name no)
@@
 			(project "Telefunken_Digitale_Electronic_101"
 				(path "/df1af5ff-c8b9-4769-9610-ead9e11e7e65/ef6275f4-75ba-4006-a847-a151b9f8c4ad"
-					(reference "C1")
+					(reference "C5")
 					(unit 1)
 				)
@@
 		(dnp no)
 		(fields_autoplaced yes)
-		(property "Reference" "C2"
+		(property "Reference" "C6"
 			(at 128.27 91.4399 0)
 			(show_name no)
@@
 			(project "Telefunken_Digitale_Electronic_101"
 				(path "/df1af5ff-c8b9-4769-9610-ead9e11e7e65/ef6275f4-75ba-4006-a847-a151b9f8c4ad"
-					(reference "C2")
+					(reference "C6")
 					(unit 1)
 				)
@@
 		(dnp no)
 		(fields_autoplaced yes)
-		(property "Reference" "#PWR07"
+		(property "Reference" "#PWR021"
 			(at 176.53 73.66 0)
 			(hide yes)
@@
 			(project "Telefunken_Digitale_Electronic_101"
 				(path "/df1af5ff-c8b9-4769-9610-ead9e11e7e65/ef6275f4-75ba-4006-a847-a151b9f8c4ad"
-					(reference "#PWR07")
+					(reference "#PWR021")
 					(unit 1)
 				)
@@
 		(dnp no)
 		(fields_autoplaced yes)
-		(property "Reference" "#PWR05"
+		(property "Reference" "#PWR017"
 			(at 116.84 97.79 0)
 			(hide yes)
@@
 			(project "Telefunken_Digitale_Electronic_101"
 				(path "/df1af5ff-c8b9-4769-9610-ead9e11e7e65/ef6275f4-75ba-4006-a847-a151b9f8c4ad"
-					(reference "#PWR05")
+					(reference "#PWR017")
 					(unit 1)
 				)
@@
 		(dnp no)
 		(fields_autoplaced yes)
-		(property "Reference" "R2"
+		(property "Reference" "R4"
 			(at 127 83.8199 0)
 			(show_name no)
@@
 			(project "Telefunken_Digitale_Electronic_101"
 				(path "/df1af5ff-c8b9-4769-9610-ead9e11e7e65/ef6275f4-75ba-4006-a847-a151b9f8c4ad"
-					(reference "R2")
+					(reference "R4")
 					(unit 1)
 				)
@@
 		(dnp no)
 		(fields_autoplaced yes)
-		(property "Reference" "#PWR01"
+		(property "Reference" "#PWR020"
 			(at 171.45 130.81 0)
 			(hide yes)
@@
 			(project "Telefunken_Digitale_Electronic_101"
 				(path "/df1af5ff-c8b9-4769-9610-ead9e11e7e65/ef6275f4-75ba-4006-a847-a151b9f8c4ad"
-					(reference "#PWR01")
+					(reference "#PWR020")
 					(unit 1)
 				)
@@
 		(dnp no)
 		(fields_autoplaced yes)
-		(property "Reference" "R1"
+		(property "Reference" "R3"
 			(at 119.38 78.7399 0)
 			(show_name no)
@@
 			(project "Telefunken_Digitale_Electronic_101"
 				(path "/df1af5ff-c8b9-4769-9610-ead9e11e7e65/ef6275f4-75ba-4006-a847-a151b9f8c4ad"
-					(reference "R1")
+					(reference "R3")
 					(unit 1)
 				)
@@
 		(dnp no)
 		(fields_autoplaced yes)
-		(property "Reference" "#PWR02"
+		(property "Reference" "#PWR016"
 			(at 116.84 80.01 0)
 			(hide yes)
@@
 			(project "Telefunken_Digitale_Electronic_101"
 				(path "/df1af5ff-c8b9-4769-9610-ead9e11e7e65/ef6275f4-75ba-4006-a847-a151b9f8c4ad"
-					(reference "#PWR02")
+					(reference "#PWR016")
 					(unit 1)
 				)
@@
 		(dnp no)
 		(fields_autoplaced yes)
-		(property "Reference" "#PWR027"
+		(property "Reference" "#PWR014"
 			(at 57.15 59.69 0)
 			(hide yes)
@@
 			(project "Telefunken_Digitale_Electronic_101"
 				(path "/df1af5ff-c8b9-4769-9610-ead9e11e7e65/ef6275f4-75ba-4006-a847-a151b9f8c4ad"
-					(reference "#PWR027")
+					(reference "#PWR014")
 					(unit 1)
 				)
@@
 		(dnp no)
 		(fields_autoplaced yes)
-		(property "Reference" "C4"
+		(property "Reference" "C8"
 			(at 191.77 71.5009 0)
 			(show_name no)
@@
 			(project "Telefunken_Digitale_Electronic_101"
 				(path "/df1af5ff-c8b9-4769-9610-ead9e11e7e65/ef6275f4-75ba-4006-a847-a151b9f8c4ad"
-					(reference "C4")
+					(reference "C8")
 					(unit 1)
 				)
@@
 		(dnp no)
 		(fields_autoplaced yes)
-		(property "Reference" "#PWR04"
+		(property "Reference" "#PWR019"
 			(at 124.46 102.87 0)
 			(hide yes)
@@
 			(project "Telefunken_Digitale_Electronic_101"
 				(path "/df1af5ff-c8b9-4769-9610-ead9e11e7e65/ef6275f4-75ba-4006-a847-a151b9f8c4ad"
-					(reference "#PWR04")
+					(reference "#PWR019")
 					(unit 1)
 				)
@@
 		(dnp no)
 		(fields_autoplaced yes)
-		(property "Reference" "#PWR06"
+		(property "Reference" "#PWR022"
 			(at 187.96 83.82 0)
 			(hide yes)
@@
 			(project "Telefunken_Digitale_Electronic_101"
 				(path "/df1af5ff-c8b9-4769-9610-ead9e11e7e65/ef6275f4-75ba-4006-a847-a151b9f8c4ad"
-					(reference "#PWR06")
-					(unit 1)
-				)
+					(reference "#PWR022")
+					(unit 1)
+				)

Commit message: adjusted connectors footprints, added footprint to input polarized capacitor, rtc and display polarized capacitors converted to non polarized
Parts:
- C8: symbol Device:C_Polarized -> Device:C
Changed lines of the file:
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@@
 	)
 	(symbol
-		(lib_id "Device:C_Polarized")
+		(lib_id "Device:C")
 		(at 187.96 73.66 0)
 		(unit 1)
@@
 		(fields_autoplaced yes)
 		(property "Reference" "C8"
-			(at 191.77 71.5009 0)
+			(at 191.77 72.3899 0)
 			(show_name no)
 			(do_not_autoplace no)
@@
 		)
 		(property "Value" "10u"
-			(at 191.77 74.0409 0)
+			(at 191.77 74.9299 0)
 			(show_name no)
 			(do_not_autoplace no)
@@
 			)
 		)
-		(property "Description" "Polarized capacitor"
+		(property "Description" "Unpolarized capacitor"
 			(at 187.96 73.66 0)
 			(hide yes)
