File: pcb/Telefunken_Digitale_Electronic_101/Telefunken_Digitale_Electronic_101.kicad_pcb (KiCad board)
At the start: 2 copper layers, 100 x 52 mm, 31 parts, among them J1 Conn_01x02_MountingPin, J2 Conn_01x02_MountingPin, J3 Conn_01x04_MountingPin, J4 Conn_01x02_Socket, J5 Conn_01x02_Socket, J6 Conn_01x02_Socket, J7 Conn_01x02_Socket, J8 Conn_01x02_Socket, SW1 SW_Push, SW2 SW_Push, U1 DS3231, U2 TM1637_SOP20

Commit message: SCH and PCB - buttons: added proper switches that will be used
Parts:
- SW1, SW2: footprint Button_Switch_THT:SW_PUSH_6mm_H4.3mm -> RadioWecker:TACT_SWITCH_3.2X4.2X2.5MM
- moved SW1 3.95 mm to (104.0, 63.0)
- moved SW2 3.95 mm to (104.0, 85.0)
Routing:
- net /Buttons/K2: track 127.0 -> 139.7 mm
- net /Buttons/K1: track 74.5 -> 67.8 mm
- net /Buttons/GRID1: track 109.5 -> 108.6 mm, vias 1 -> 0
- net GND: vias 62 -> 70
