File: pcb/Core_PCB/display.kicad_sch (KiCad schematic)
At the start: 4 parts, among them J4 Conn_01x02_MountingPin, J5 Conn_01x02_MountingPin, J6 Conn_01x04_MountingPin

Commit message: SCH: annotated sheets, reannotated all components
Parts:
- J3: renamed from J5; Name Display -> DISPLAY
- renumbered C2 to C3, J4 to J2, J6 to J4
Other:
- company: (none) -> brunolalb@gmail.com
- title: (none) -> Alarm Clock Resto Mod - Core PCB
Changed lines of the file:
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@@
 	(generator_version "10.0")
 	(paper "A4")
+	(title_block
+		(title "Alarm Clock Resto Mod - Core PCB")
+		(date "2026-07-08")
+		(rev "1.0")
+		(company "brunolalb@gmail.com")
+		(comment 1 "Bruno Landau Albrecht")
+	)
 	(junction
 		(at 107.95 63.5)
@@
 		(dnp no)
 		(fields_autoplaced yes)
-		(property "Reference" "#PWR07"
+		(property "Reference" "#PWR016"
 			(at 163.83 77.47 0)
 			(hide yes)
@@
 			(project "Core_PCB"
 				(path "/79975d02-cfea-4cc3-8869-9743c86248b2/00b4dbc5-1324-45e9-962d-9bcf13f06c40"
-					(reference "#PWR07")
+					(reference "#PWR016")
 					(unit 1)
 				)
@@
 		(dnp no)
 		(fields_autoplaced yes)
-		(property "Reference" "#PWR045"
+		(property "Reference" "#PWR012"
 			(at 107.95 59.69 0)
 			(hide yes)
@@
 			(project "Core_PCB"
 				(path "/79975d02-cfea-4cc3-8869-9743c86248b2/00b4dbc5-1324-45e9-962d-9bcf13f06c40"
-					(reference "#PWR045")
+					(reference "#PWR012")
 					(unit 1)
 				)
@@
 		(dnp no)
 		(fields_autoplaced yes)
-		(property "Reference" "C2"
+		(property "Reference" "C3"
 			(at 115.57 58.4199 0)
 			(show_name no)
@@
 			(project "Core_PCB"
 				(path "/79975d02-cfea-4cc3-8869-9743c86248b2/00b4dbc5-1324-45e9-962d-9bcf13f06c40"
-					(reference "C2")
+					(reference "C3")
 					(unit 1)
 				)
@@
 		(dnp no)
 		(fields_autoplaced yes)
-		(property "Reference" "#PWR023"
+		(property "Reference" "#PWR015"
 			(at 92.71 74.93 0)
 			(hide yes)
@@
 			(project "Core_PCB"
 				(path "/79975d02-cfea-4cc3-8869-9743c86248b2/00b4dbc5-1324-45e9-962d-9bcf13f06c40"
-					(reference "#PWR023")
+					(reference "#PWR015")
 					(unit 1)
 				)
@@
 		(dnp no)
 		(fields_autoplaced yes)
-		(property "Reference" "#PWR02"
+		(property "Reference" "#PWR018"
 			(at 96.52 129.54 0)
 			(hide yes)
@@
 			(project "Core_PCB"
 				(path "/79975d02-cfea-4cc3-8869-9743c86248b2/00b4dbc5-1324-45e9-962d-9bcf13f06c40"
-					(reference "#PWR02")
+					(reference "#PWR018")
 					(unit 1)
 				)
@@
 		(in_pos_files yes)
 		(dnp no)
-		(property "Reference" "J6"
+		(property "Reference" "J4"
 			(at 96.52 104.14 0)
 			(hide yes)
@@
 			(project "Core_PCB"
 				(path "/79975d02-cfea-4cc3-8869-9743c86248b2/00b4dbc5-1324-45e9-962d-9bcf13f06c40"
-					(reference "J6")
+					(reference "J4")
 					(unit 1)
 				)
@@
 		(in_pos_files yes)
 		(dnp no)
-		(property "Reference" "J4"
+		(property "Reference" "J2"
 			(at 92.71 54.61 0)
 			(hide yes)
@@
 			(project "Core_PCB"
 				(path "/79975d02-cfea-4cc3-8869-9743c86248b2/00b4dbc5-1324-45e9-962d-9bcf13f06c40"
-					(reference "J4")
+					(reference "J2")
 					(unit 1)
 				)
@@
 		(dnp no)
 		(fields_autoplaced yes)
-		(property "Reference" "#PWR04"
+		(property "Reference" "#PWR013"
 			(at 107.95 69.85 0)
 			(hide yes)
@@
 			(project "Core_PCB"
 				(path "/79975d02-cfea-4cc3-8869-9743c86248b2/00b4dbc5-1324-45e9-962d-9bcf13f06c40"
-					(reference "#PWR04")
+					(reference "#PWR013")
 					(unit 1)
 				)
@@
 		(dnp no)
 		(fields_autoplaced yes)
-		(property "Reference" "#PWR06"
+		(property "Reference" "#PWR014"
 			(at 163.83 71.12 0)
 			(hide yes)
@@
 			(project "Core_PCB"
 				(path "/79975d02-cfea-4cc3-8869-9743c86248b2/00b4dbc5-1324-45e9-962d-9bcf13f06c40"
-					(reference "#PWR06")
+					(reference "#PWR014")
 					(unit 1)
 				)
@@
 		(in_pos_files yes)
 		(dnp no)
-		(property "Reference" "J5"
+		(property "Reference" "J3"
 			(at 96.52 81.28 0)
 			(hide yes)
@@
 			)
 		)
-		(property "Name" "Display"
+		(property "Name" "DISPLAY"
 			(at 96.774 81.534 0)
 			(show_name no)
@@
 			(project "Core_PCB"
 				(path "/79975d02-cfea-4cc3-8869-9743c86248b2/00b4dbc5-1324-45e9-962d-9bcf13f06c40"
-					(reference "J5")
+					(reference "J3")
 					(unit 1)
 				)
@@
 		(dnp no)
 		(fields_autoplaced yes)
-		(property "Reference" "#PWR01"
+		(property "Reference" "#PWR017"
 			(at 96.52 101.6 0)
 			(hide yes)
@@
 			(project "Core_PCB"
 				(path "/79975d02-cfea-4cc3-8869-9743c86248b2/00b4dbc5-1324-45e9-962d-9bcf13f06c40"
-					(reference "#PWR01")
+					(reference "#PWR017")
 					(unit 1)
 				)

Commit message: SCH: assigned footprints to what had missing, replaced some polarized caps with non polarized, added connector for capacitance sensor, ran electric test and fixed minor issues
Changed lines of the file:
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@@
 		)
 	)
-	(hierarchical_label "3V3"
+	(hierarchical_label "+3V3"
 		(shape bidirectional)
 		(at 166.37 67.31 0)
