File: pcb/Core_PCB/sdcard.kicad_sch (KiCad schematic)
At the start: 1 part, among them J3 Conn_01x06

Commit message: SCH: annotated sheets, reannotated all components
Parts:
- J5: renamed from J3; Name (none) -> SDCARD
Other:
- company: (none) -> brunolalb@gmail.com
- title: (none) -> Alarm Clock Resto Mod - Core PCB
Changed lines of the file:
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@@
 	(generator_version "10.0")
 	(paper "A4")
+	(title_block
+		(title "Alarm Clock Resto Mod - Core PCB")
+		(date "2026-07-08")
+		(rev "1.0")
+		(company "brunolalb@gmail.com")
+		(comment 1 "Bruno Landau Albrecht")
+	)
 	(wire
 		(pts
@@
 		(dnp no)
 		(fields_autoplaced yes)
-		(property "Reference" "#PWR034"
+		(property "Reference" "#PWR020"
 			(at 76.2 48.26 0)
 			(hide yes)
@@
 			(project "Core_PCB"
 				(path "/79975d02-cfea-4cc3-8869-9743c86248b2/19a27239-6385-4c28-86b1-a5a9f657999b"
-					(reference "#PWR034")
+					(reference "#PWR020")
 					(unit 1)
 				)
@@
 		(dnp no)
 		(fields_autoplaced yes)
-		(property "Reference" "#PWR033"
+		(property "Reference" "#PWR019"
 			(at 76.2 41.91 0)
 			(hide yes)
@@
 			(project "Core_PCB"
 				(path "/79975d02-cfea-4cc3-8869-9743c86248b2/19a27239-6385-4c28-86b1-a5a9f657999b"
-					(reference "#PWR033")
+					(reference "#PWR019")
 					(unit 1)
 				)
@@
 		(dnp no)
 		(fields_autoplaced yes)
-		(property "Reference" "#PWR031"
+		(property "Reference" "#PWR021"
 			(at 119.38 45.72 0)
 			(hide yes)
@@
 			(project "Core_PCB"
 				(path "/79975d02-cfea-4cc3-8869-9743c86248b2/19a27239-6385-4c28-86b1-a5a9f657999b"
-					(reference "#PWR031")
+					(reference "#PWR021")
 					(unit 1)
 				)
@@
 		(in_pos_files yes)
 		(dnp no)
-		(fields_autoplaced yes)
-		(property "Reference" "J3"
+		(property "Reference" "J5"
 			(at 109.22 35.56 0)
 			(show_name no)
@@
 			(at 109.22 46.99 0)
 			(hide yes)
+			(show_name no)
+			(do_not_autoplace no)
+			(effects
+				(font
+					(size 1.27 1.27)
+				)
+			)
+		)
+		(property "Name" "SDCARD"
+			(at 107.95 58.42 0)
 			(show_name no)
 			(do_not_autoplace no)
@@
 			(project "Core_PCB"
 				(path "/79975d02-cfea-4cc3-8869-9743c86248b2/19a27239-6385-4c28-86b1-a5a9f657999b"
-					(reference "J3")
+					(reference "J5")
 					(unit 1)
 				)
@@
 		(dnp no)
 		(fields_autoplaced yes)
-		(property "Reference" "#PWR032"
+		(property "Reference" "#PWR022"
 			(at 114.3 60.96 0)
 			(hide yes)
@@
 			(project "Core_PCB"
 				(path "/79975d02-cfea-4cc3-8869-9743c86248b2/19a27239-6385-4c28-86b1-a5a9f657999b"
-					(reference "#PWR032")
+					(reference "#PWR022")
 					(unit 1)
 				)

Commit message: SCH: assigned footprints to what had missing, replaced some polarized caps with non polarized, added connector for capacitance sensor, ran electric test and fixed minor issues
Parts:
- J5: footprint (none) -> Connector_PinSocket_2.54mm:PinSocket_1x06_P2.54mm_Vertical
Changed lines of the file:
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@@
 		)
 	)
-	(hierarchical_label "3V3"
+	(hierarchical_label "+3V3"
 		(shape bidirectional)
 		(at 78.74 38.1 0)
@@
 			)
 		)
-		(property "Footprint" ""
+		(property "Footprint" "Connector_PinSocket_2.54mm:PinSocket_1x06_P2.54mm_Vertical"
 			(at 109.22 46.99 0)
 			(hide yes)
