File: pcb/Core_PCB/Core_PCB.kicad_pcb (KiCad board)
At the start: 2 copper layers, 60 x 110 mm, 68 parts, among them J1 Conn_01x02_MountingPin, J10 Conn_02x12_Odd_Even, J11 Conn_01x03_MountingPin, J2 Conn_01x02_MountingPin, J3 Conn_01x02_MountingPin, J4 Conn_01x04_MountingPin, J5 Conn_01x06, J6 Screw_Terminal_01x02, J7 Conn_01x02_MountingPin, J8 Conn_01x08, J9 Conn_01x08, Q1 BSN20, SW1 SW_Push, SW2 SW_Push, SW3 SW_Push, U1 MAX98357A, U2 HEF4051BT, U3 MPR121_BREAKOUT, U4 MCP23017x-x-SS

Commit message: PCBs: updated logo; added I2C resistors to I2C (core pcb)
Parts:
- removed LF1: ~, RadioWecker:LEAF
- added G1: LOGO, RadioWecker:LOGO, F.Cu at (153.5, 78.6)
- added R20: 2K2, Resistor_SMD:R_0603_1608Metric_Pad0.98x0.95mm_HandSolder, B.Cu at (128.5, 87.6)
- added R21: 2K2, Resistor_SMD:R_0603_1608Metric_Pad0.98x0.95mm_HandSolder, B.Cu at (127.6, 83.6)
